File: hw/kanelbulle.sch (KiCad schematic (older format))
At the start: 83 parts, among them J1 USB, U1 LPC1114/302, U2 PCA9685, U3 ULN2003A, U4 ULN2003A, U5 ULN2003A

Commit message: decoupling
Parts:
- gave numbers to parts that had none: 7
Changed lines of the file:
@@
 	11700 18500 10600 18500
 $Comp
-L 3V3 #PWR01
+L 3V3 #PWR4
 U 1 1 54CFB406
 P 20100 2350
-F 0 "#PWR01" H 20100 2450 40  0001 C CNN
+F 0 "#PWR4" H 20100 2450 40  0001 C CNN
 F 1 "3V3" H 20100 2475 40  0000 C CNN
 F 2 "" H 20100 2350 60  0000 C CNN
@@
 $EndComp
 $Comp
-L 3V3 #PWR02
+L 3V3 #PWR5
 U 1 1 54CFB413
 P 22350 2350
-F 0 "#PWR02" H 22350 2450 40  0001 C CNN
+F 0 "#PWR5" H 22350 2450 40  0001 C CNN
 F 1 "3V3" H 22350 2475 40  0000 C CNN
 F 2 "" H 22350 2350 60  0000 C CNN
@@
 $EndComp
 $Comp
-L 3V3 #PWR03
+L 3V3 #PWR6
 U 1 1 54CFB419
 P 24250 2350
-F 0 "#PWR03" H 24250 2450 40  0001 C CNN
+F 0 "#PWR6" H 24250 2450 40  0001 C CNN
 F 1 "3V3" H 24250 2475 40  0000 C CNN
 F 2 "" H 24250 2350 60  0000 C CNN
@@
 $EndComp
 $Comp
-L 3V3 #PWR04
+L 3V3 #PWR7
 U 1 1 54CFB41F
 P 26100 2350
-F 0 "#PWR04" H 26100 2450 40  0001 C CNN
+F 0 "#PWR7" H 26100 2450 40  0001 C CNN
 F 1 "3V3" H 26100 2475 40  0000 C CNN
 F 2 "" H 26100 2350 60  0000 C CNN
@@
 $EndComp
 $Comp
-L 3V3 #PWR05
+L 3V3 #PWR8
 U 1 1 54CFB425
 P 28050 2350
-F 0 "#PWR05" H 28050 2450 40  0001 C CNN
+F 0 "#PWR8" H 28050 2450 40  0001 C CNN
 F 1 "3V3" H 28050 2475 40  0000 C CNN
 F 2 "" H 28050 2350 60  0000 C CNN
@@
 Connection ~ 8150 16800
 $Comp
-L 3V3 #PWR06
+L 3V3 #PWR10
 U 1 1 54CFC851
 P 8150 16650
-F 0 "#PWR06" H 8150 16750 40  0001 C CNN
+F 0 "#PWR10" H 8150 16750 40  0001 C CNN
 F 1 "3V3" H 8150 16775 40  0000 C CNN
 F 2 "" H 8150 16650 60  0000 C CNN
@@
 $EndComp
 $Comp
-L GND #PWR07
+L GND #PWR11
 U 1 1 54CFC924
 P 8750 19100
-F 0 "#PWR07" H 8750 19100 30  0001 C CNN
+F 0 "#PWR11" H 8750 19100 30  0001 C CNN
 F 1 "GND" H 8750 19030 30  0001 C CNN
 F 2 "" H 8750 19100 60  0000 C CNN
@@
 	5950 2100 6050 2100
 $Comp
-L GND #PWR08
+L GND #PWR3
 U 1 1 54CFDFE0
 P 5450 2150
-F 0 "#PWR08" H 5450 2150 30  0001 C CNN
+F 0 "#PWR3" H 5450 2150 30  0001 C CNN
 F 1 "GND" H 5450 2080 30  0001 C CNN
 F 2 "" H 5450 2150 60  0000 C CNN
@@
 $EndComp
 $Comp
-L 3V3 #PWR09
+L 3V3 #PWR1
 U 1 1 54CFDFEF
 P 6000 1700
-F 0 "#PWR09" H 6000 1800 40  0001 C CNN
+F 0 "#PWR1" H 6000 1800 40  0001 C CNN
 F 1 "3V3" H 6000 1825 40  0000 C CNN
 F 2 "" H 6000 1700 60  0000 C CNN
@@
 TX
 $Comp
-L C C?
+L C C2
 U 1 1 54CFB5F9
 P 10600 2300
-F 0 "C?" H 10600 2400 40  0000 L CNN
+F 0 "C2" H 10600 2400 40  0000 L CNN
 F 1 "C" H 10606 2215 40  0000 L CNN
 F 2 "~" H 10638 2150 30  0000 C CNN
@@
 $EndComp
 $Comp
-L C C?
+L C C3
 U 1 1 54CFB606
 P 10800 2300
-F 0 "C?" H 10800 2400 40  0000 L CNN
+F 0 "C3" H 10800 2400 40  0000 L CNN
 F 1 "C" H 10806 2215 40  0000 L CNN
 F 2 "~" H 10838 2150 30  0000 C CNN
@@
 $EndComp
 $Comp
-L C C?
+L C C4
 U 1 1 54CFB60C
 P 11000 2300
-F 0 "C?" H 11000 2400 40  0000 L CNN
+F 0 "C4" H 11000 2400 40  0000 L CNN
 F 1 "C" H 11006 2215 40  0000 L CNN
 F 2 "~" H 11038 2150 30  0000 C CNN
@@
 $EndComp
 $Comp
-L C C?
+L C C5
 U 1 1 54CFB612
 P 11200 2300
-F 0 "C?" H 11200 2400 40  0000 L CNN
+F 0 "C5" H 11200 2400 40  0000 L CNN
 F 1 "C" H 11206 2215 40  0000 L CNN
 F 2 "~" H 11238 2150 30  0000 C CNN
@@
 $EndComp
 $Comp
-L C C?
+L C C6
 U 1 1 54CFB618
 P 11400 2300
-F 0 "C?" H 11400 2400 40  0000 L CNN
+F 0 "C6" H 11400 2400 40  0000 L CNN
 F 1 "C" H 11406 2215 40  0000 L CNN
 F 2 "~" H 11438 2150 30  0000 C CNN
@@
 $EndComp
 $Comp
-L C C?
+L C C7
 U 1 1 54CFB61E
 P 11600 2300
-F 0 "C?" H 11600 2400 40  0000 L CNN
+F 0 "C7" H 11600 2400 40  0000 L CNN
 F 1 "C" H 11606 2215 40  0000 L CNN
 F 2 "~" H 11638 2150 30  0000 C CNN
@@
 $EndComp
 $Comp
-L C C?
+L C C1
 U 1 1 54CFB624
 P 10400 2300
-F 0 "C?" H 10400 2400 40  0000 L CNN
+F 0 "C1" H 10400 2400 40  0000 L CNN
 F 1 "C" H 10406 2215 40  0000 L CNN
 F 2 "~" H 10438 2150 30  0000 C CNN
@@
 Connection ~ 11400 2500
 $Comp
-L GND #PWR?
+L GND #PWR9
 U 1 1 54CFCF5E
 P 11000 2600
-F 0 "#PWR?" H 11000 2600 30  0001 C CNN
+F 0 "#PWR9" H 11000 2600 30  0001 C CNN
 F 1 "GND" H 11000 2530 30  0001 C CNN
 F 2 "" H 11000 2600 60  0000 C CNN
@@
 	11000 2600 11000 2500
 $Comp
-L 3V3 #PWR?
+L 3V3 #PWR2
 U 1 1 54CFD18D
 P 11000 2000
-F 0 "#PWR?" H 11000 2100 40  0001 C CNN
+F 0 "#PWR2" H 11000 2100 40  0001 C CNN
 F 1 "3V3" H 11000 2125 40  0000 C CNN
 F 2 "" H 11000 2000 60  0000 C CNN

Commit message: aaawww yeeeeaaaahhhh
Parts:
- removed J1: USB, symbol USB
- added C8: C, ~, symbol C
- added P1: USB, symbol CONN_4
- added P2: CONN_6, symbol CONN_6
- added U6: NCP1117ST33T3G, symbol NCP1117ST33T3G
Connections:
- net labels added: +5V, LEDOE
- wire segments 326 -> 357
- no-connect marks 0 -> 12
