File: hw/kanelbulle.sch (KiCad schematic (older format))
At the start: 86 parts, among them P1 USB, P2 CONN_6, U1 LPC1114/302, U2 PCA9685, U3 ULN2003A, U4 ULN2003A, U5 ULN2003A, U6 NCP1117ST33T3G

Commit message: gerber plot
Connections:
- no-connect marks 12 -> 49
Changed lines of the file:
@@
 	11700 18500 10600 18500
 $Comp
-L 3V3 #PWR21
+L 3V3 #PWR01
 U 1 1 54CFB406
 P 20100 2350
-F 0 "#PWR21" H 20100 2450 40  0001 C CNN
+F 0 "#PWR01" H 20100 2450 40  0001 C CNN
 F 1 "3V3" H 20100 2475 40  0000 C CNN
 F 2 "" H 20100 2350 60  0000 C CNN
@@
 $EndComp
 $Comp
-L 3V3 #PWR22
+L 3V3 #PWR02
 U 1 1 54CFB413
 P 22350 2350
-F 0 "#PWR22" H 22350 2450 40  0001 C CNN
+F 0 "#PWR02" H 22350 2450 40  0001 C CNN
 F 1 "3V3" H 22350 2475 40  0000 C CNN
 F 2 "" H 22350 2350 60  0000 C CNN
@@
 $EndComp
 $Comp
-L 3V3 #PWR23
+L 3V3 #PWR03
 U 1 1 54CFB419
 P 24250 2350
-F 0 "#PWR23" H 24250 2450 40  0001 C CNN
+F 0 "#PWR03" H 24250 2450 40  0001 C CNN
 F 1 "3V3" H 24250 2475 40  0000 C CNN
 F 2 "" H 24250 2350 60  0000 C CNN
@@
 $EndComp
 $Comp
-L 3V3 #PWR24
+L 3V3 #PWR04
 U 1 1 54CFB41F
 P 26100 2350
-F 0 "#PWR24" H 26100 2450 40  0001 C CNN
+F 0 "#PWR04" H 26100 2450 40  0001 C CNN
 F 1 "3V3" H 26100 2475 40  0000 C CNN
 F 2 "" H 26100 2350 60  0000 C CNN
@@
 $EndComp
 $Comp
-L 3V3 #PWR25
+L 3V3 #PWR05
 U 1 1 54CFB425
 P 28050 2350
-F 0 "#PWR25" H 28050 2450 40  0001 C CNN
+F 0 "#PWR05" H 28050 2450 40  0001 C CNN
 F 1 "3V3" H 28050 2475 40  0000 C CNN
 F 2 "" H 28050 2350 60  0000 C CNN
@@
 Connection ~ 8150 16800
 $Comp
-L 3V3 #PWR5
+L 3V3 #PWR06
 U 1 1 54CFC851
 P 8150 16650
-F 0 "#PWR5" H 8150 16750 40  0001 C CNN
+F 0 "#PWR06" H 8150 16750 40  0001 C CNN
 F 1 "3V3" H 8150 16775 40  0000 C CNN
 F 2 "" H 8150 16650 60  0000 C CNN
@@
 $EndComp
 $Comp
-L GND #PWR8
+L GND #PWR07
 U 1 1 54CFC924
 P 8750 19100
-F 0 "#PWR8" H 8750 19100 30  0001 C CNN
+F 0 "#PWR07" H 8750 19100 30  0001 C CNN
 F 1 "GND" H 8750 19030 30  0001 C CNN
 F 2 "" H 8750 19100 60  0000 C CNN
@@
 	5950 2100 6050 2100
 $Comp
-L GND #PWR3
+L GND #PWR08
 U 1 1 54CFDFE0
 P 5450 2150
-F 0 "#PWR3" H 5450 2150 30  0001 C CNN
+F 0 "#PWR08" H 5450 2150 30  0001 C CNN
 F 1 "GND" H 5450 2080 30  0001 C CNN
 F 2 "" H 5450 2150 60  0000 C CNN
@@
 $EndComp
 $Comp
-L 3V3 #PWR4
+L 3V3 #PWR09
 U 1 1 54CFDFEF
 P 6000 1700
-F 0 "#PWR4" H 6000 1800 40  0001 C CNN
+F 0 "#PWR09" H 6000 1800 40  0001 C CNN
 F 1 "3V3" H 6000 1825 40  0000 C CNN
 F 2 "" H 6000 1700 60  0000 C CNN
@@
 Connection ~ 11400 2500
 $Comp
-L GND #PWR12
+L GND #PWR010
 U 1 1 54CFCF5E
 P 11000 2600
-F 0 "#PWR12" H 11000 2600 30  0001 C CNN
+F 0 "#PWR010" H 11000 2600 30  0001 C CNN
 F 1 "GND" H 11000 2530 30  0001 C CNN
 F 2 "" H 11000 2600 60  0000 C CNN
@@
 	11000 2600 11000 2500
 $Comp
-L 3V3 #PWR11
+L 3V3 #PWR011
 U 1 1 54CFD18D
 P 11000 2000
-F 0 "#PWR11" H 11000 2100 40  0001 C CNN
+F 0 "#PWR011" H 11000 2100 40  0001 C CNN
 F 1 "3V3" H 11000 2125 40  0000 C CNN
 F 2 "" H 11000 2000 60  0000 C CNN
@@
 $EndComp
 $Comp
-L GND #PWR16
+L GND #PWR012
 U 1 1 54D0A630
 P 12100 4700
-F 0 "#PWR16" H 12100 4700 30  0001 C CNN
+F 0 "#PWR012" H 12100 4700 30  0001 C CNN
 F 1 "GND" H 12100 4630 30  0001 C CNN
 F 2 "" H 12100 4700 60  0000 C CNN
@@
 $EndComp
 $Comp
-L 3V3 #PWR20
+L 3V3 #PWR013
 U 1 1 54D0A63F
 P 12550 4300
-F 0 "#PWR20" H 12550 4400 40  0001 C CNN
+F 0 "#PWR013" H 12550 4400 40  0001 C CNN
 F 1 "3V3" H 12550 4425 40  0000 C CNN
 F 2 "" H 12550 4300 60  0000 C CNN
@@
 	12100 4700 12100 4650
 $Comp
-L +5V #PWR15
+L +5V #PWR014
 U 1 1 54D0AA95
 P 11650 4300
-F 0 "#PWR15" H 11650 4390 20  0001 C CNN
+F 0 "#PWR014" H 11650 4390 20  0001 C CNN
 F 1 "+5V" H 11650 4390 30  0000 C CNN
 F 2 "" H 11650 4300 60  0000 C CNN
@@
 $EndComp
 $Comp
-L +5V #PWR13
+L +5V #PWR015
 U 1 1 54D0ACD7
 P 11250 4300
-F 0 "#PWR13" H 11250 4390 20  0001 C CNN
+F 0 "#PWR015" H 11250 4390 20  0001 C CNN
 F 1 "+5V" H 11250 4390 30  0000 C CNN
 F 2 "" H 11250 4300 60  0000 C CNN
@@
 $EndComp
 $Comp
-L GND #PWR14
+L GND #PWR016
 U 1 1 54D0ACDD
 P 11250 4800
-F 0 "#PWR14" H 11250 4800 30  0001 C CNN
+F 0 "#PWR016" H 11250 4800 30  0001 C CNN
 F 1 "GND" H 11250 4730 30  0001 C CNN
 F 2 "" H 11250 4800 60  0000 C CNN
@@
 $EndComp
 $Comp
-L +5V #PWR10
+L +5V #PWR017
 U 1 1 54D0B23D
 P 9750 4150
-F 0 "#PWR10" H 9750 4240 20  0001 C CNN
+F 0 "#PWR017" H 9750 4240 20  0001 C CNN
 F 1 "+5V" H 9750 4240 30  0000 C CNN
 F 2 "" H 9750 4150 60  0000 C CNN
@@
 $EndComp
 $Comp
-L GND #PWR9
+L GND #PWR018
 U 1 1 54D0B243
 P 9350 4250
-F 0 "#PWR9" H 9350 4250 30  0001 C CNN
+F 0 "#PWR018" H 9350 4250 30  0001 C CNN
 F 1 "GND" H 9350 4180 30  0001 C CNN
 F 2 "" H 9350 4250 60  0000 C CNN
@@
 RST
 $Comp
-L 3V3 #PWR1
+L 3V3 #PWR019
 U 1 1 54D0CBC6
 P 2050 3250
-F 0 "#PWR1" H 2050 3350 40  0001 C CNN
+F 0 "#PWR019" H 2050 3350 40  0001 C CNN
 F 1 "3V3" H 2050 3375 40  0000 C CNN
 F 2 "" H 2050 3250 60  0000 C CNN
@@
 $EndComp
 $Comp
-L GND #PWR2
+L GND #PWR020
 U 1 1 54D0CBD5
 P 2050 3350
-F 0 "#PWR2" H 2050 3350 30  0001 C CNN
+F 0 "#PWR020" H 2050 3350 30  0001 C CNN
 F 1 "GND" H 2050 3280 30  0001 C CNN
 F 2 "" H 2050 3350 60  0000 C CNN
@@
 Connection ~ 12450 17200
 $Comp
-L GND #PWR17
+L GND #PWR021
 U 1 1 54D0D146
 P 12450 17300
-F 0 "#PWR17" H 12450 17300 30  0001 C CNN
+F 0 "#PWR021" H 12450 17300 30  0001 C CNN
 F 1 "GND" H 12450 17230 30  0001 C CNN
 F 2 "" H 12450 17300 60  0000 C CNN
@@
 Connection ~ 12450 19400
 $Comp
-L GND #PWR18
+L GND #PWR022
 U 1 1 54D0DA29
 P 12450 18400
-F 0 "#PWR18" H 12450 18400 30  0001 C CNN
+F 0 "#PWR022" H 12450 18400 30  0001 C CNN
 F 1 "GND" H 12450 18330 30  0001 C CNN
 F 2 "" H 12450 18400 60  0000 C CNN
@@
 $EndComp
 $Comp
-L GND #PWR19
+L GND #PWR023
 U 1 1 54D0DA38
 P 12450 19500
-F 0 "#PWR19" H 12450 19500 30  0001 C CNN
+F 0 "#PWR023" H 12450 19500 30  0001 C CNN
 F 1 "GND" H 12450 19430 30  0001 C CNN
 F 2 "" H 12450 19500 60  0000 C CNN
@@
 Connection ~ 8700 17900
 $Comp
-L GND #PWR7
+L GND #PWR024
 U 1 1 54D0E66C
 P 8700 18150
-F 0 "#PWR7" H 8700 18150 30  0001 C CNN
+F 0 "#PWR024" H 8700 18150 30  0001 C CNN
 F 1 "GND" H 8700 18080 30  0001 C CNN
 F 2 "" H 8700 18150 60  0000 C CNN
@@
 Connection ~ 8600 17800
 $Comp
-L 3V3 #PWR6
+L 3V3 #PWR025
 U 1 1 54D0ED3D
 P 8600 17550
-F 0 "#PWR6" H 8600 17650 40  0001 C CNN
+F 0 "#PWR025" H 8600 17650 40  0001 C CNN
 F 1 "3V3" H 8600 17675 40  0000 C CNN
 F 2 "" H 8600 17550 60  0000 C CNN
@@
 	5450 2050 5450 2150
 Connection ~ 5700 2100
+NoConn ~ 4900 2850
+NoConn ~ 4900 3250
+NoConn ~ 4900 3350
+NoConn ~ 4900 3450
+NoConn ~ 4900 3550
+NoConn ~ 4900 3650
+NoConn ~ 4900 3750
+NoConn ~ 4900 4350
+NoConn ~ 4900 4450
+NoConn ~ 4900 4550
+NoConn ~ 4900 4650
+NoConn ~ 4900 4750
+NoConn ~ 4900 4850
+NoConn ~ 4900 5150
+NoConn ~ 4900 5250
+NoConn ~ 4900 5350
+NoConn ~ 4900 5450
+NoConn ~ 6750 4350
+NoConn ~ 6750 4450
+NoConn ~ 6750 4550
+NoConn ~ 6750 4650
+NoConn ~ 6750 4750
+NoConn ~ 6750 4850
+NoConn ~ 6750 4950
+NoConn ~ 6750 5050
+NoConn ~ 6750 5150
+NoConn ~ 6750 5250
+NoConn ~ 6750 5350
+NoConn ~ 6750 5450
+NoConn ~ 6750 2650
+NoConn ~ 6750 2750
+NoConn ~ 6750 2850
+NoConn ~ 6750 2950
+NoConn ~ 6750 3050
+NoConn ~ 6750 3150
+NoConn ~ 5750 5950
+NoConn ~ 5950 5950
 $EndSCHEMATC
