File: hw/kanelbulle.kicad_pcb (KiCad board)
At the start: 2 copper layers, 50 x 50 mm, 86 parts, among them P1 USB, P2 CONN_6, U1 LPC1114/302, U2 PCA9685, U3 ULN2003A, U4 ULN2003A, U5 ULN2003A, U6 NCP1117ST33T3G

Commit message: gerber plot
Parts:
- added G***: LOGO, LOGO, B.Cu at (188.3, 164.2)
Routing:
- net GND: track 13.4 -> 16.1 mm
Other:
- board text added: "2015, MIT License"
- board text added: "Alex Wennberg"
- board text added: "Axel Isaksson"
- board text added: "Kanelbulle"
- board text added: "Rickard Eriksson"
- board text added: "Sajjadali Hemani"
- board text added: "Steven Arnow"
